File: power-board/power-board.kicad_pcb (KiCad board)
At the start: 4 copper layers, 90 x 70 mm, 133 parts, among them J1001 PA[5..7], J1002 PB[0..3], J1101 USB_OTG, J1102 CSHARE_IN, J1103 CSHARE_OUT, J301 CONN_01X02, J601 PDI, J801 CONN_02X05, J901 CONN_01X04, J902 CONN_01X04, J903 CONN_01X04, J904 CONN_01X04, J905 CONN_01X04, J906 PC[0..1], Q301 Q_NMOS_SSSGD, SW601 RESET, U1101 TPD2E001IDRLRQ1, U201 LMZ23610, U301 RT1720, U401 TLV521, U501 3.3v, U601 ATXMEGA32A4U-AU, U701 Main Reg, U901 CD4504B, Y601 16MHz

Commit message: finished up parts ordering and generated gerbers
Other:
- rule pad_to_mask_clearance: 0.2 -> 0
Changed lines of the file:
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@@
-(kicad_pcb (version 4) (host pcbnew 4.0.6)
+(kicad_pcb (version 4) (host pcbnew 4.0.7)
   (general
     (links 590)
@@
     (pad_size 1.7 1.7)
     (pad_drill 1)
-    (pad_to_mask_clearance 0.2)
+    (pad_to_mask_clearance 0)
     (aux_axis_origin 0 0)
     (visible_elements FFFFFF7F)
     (pcbplotparams
-      (layerselection 0x00030_80000001)
-      (usegerberextensions false)
+      (layerselection 0x011a8_80000007)
+      (usegerberextensions true)
       (excludeedgelayer true)
       (linewidth 0.100000)
@@
       (outputformat 1)
       (mirror false)
-      (drillshape 1)
+      (drillshape 0)
       (scaleselection 1)
-      (outputdirectory ""))
+      (outputdirectory gerbers))
   )
   (net 0 "")
